Commit message: joystick&slam

File: description/lidar.xacro (robot description, xacro)
@@ -4,5 +4,5 @@
         <parent link="chassis"/>
         <child link="laser_frame"/>
-        <origin xyz="0.1 0 0.175" rpy="0 0 0"/>
+        <origin xyz="0.1 0 0.075" rpy="0 0 0"/>
     </joint>
     <link name="laser_frame">

File: description/robot_core.xacro (robot description, xacro)
@@ -20,4 +20,12 @@
     <link name="base_link">
     </link>
+    <!-- BASE_FOOTPRINT LINK -->
+    <joint name="base_footprint_joint" type="fixed">
+        <parent link="base_link"/>
+        <child link="base_footprint"/>
+        <origin xyz="0 0 0" rpy="0 0 0"/>
+    </joint>
+    <link name="base_footprint">
+    </link>
     <!-- CHASSIS LINK -->
     <joint name="chassis_joint" type="fixed">
@@ -28,18 +36,18 @@
     <link name="chassis">
         <visual>
-            <origin xyz="0.15 0 0.075"/>
+            <origin xyz="0.15 0 0.05"/>
             <geometry>
-                <box size="0.3 0.3 0.15"/>
+                <box size="0.23 0.3 0.05"/>
             </geometry>
             <material name="white"/>
         </visual>
         <collision>
-            <origin xyz="0.15 0 0.075"/>
+            <origin xyz="0.15 0 0.05"/>
             <geometry>
-                <box size="0.3 0.3 0.15"/>
+                <box size="0.23 0.3 0.05"/>
             </geometry>
         </collision>
         <xacro:inertial_box mass="0.5" x="0.3" y="0.3" z="0.15">
-            <origin xyz="0.15 0 0.075" rpy="0 0 0"/>
+            <origin xyz="0.15 0 0.05" rpy="0 0 0"/>
         </xacro:inertial_box>
     </link>
@@ -51,5 +59,5 @@
         <parent link="base_link"/>
         <child link="left_wheel"/>
-        <origin xyz="0 0.175 0" rpy="-${pi/2} 0 0" />
+        <origin xyz="0 0.175 -0.02" rpy="-${pi/2} 0 0" />
         <axis xyz="0 0 1"/>
     </joint>
@@ -57,5 +65,5 @@
         <visual>
             <geometry>
-                <cylinder radius="0.05" length="0.04"/>
+                <cylinder radius="0.031" length="0.025"/>
             </geometry>
             <material name="blue"/>
@@ -63,5 +71,5 @@
         <collision>
             <geometry>
-                <sphere radius="0.05"/>
+                <sphere radius="0.031"/>
             </geometry>
         </collision>
@@ -77,5 +85,5 @@
         <parent link="base_link"/>
         <child link="right_wheel"/>
-        <origin xyz="0 -0.175 0" rpy="${pi/2} 0 0" />
+        <origin xyz="0 -0.175 -0.02" rpy="${pi/2} 0 0" />
         <axis xyz="0 0 -1"/>
     </joint>
@@ -83,5 +91,5 @@
         <visual>
             <geometry>
-                <cylinder radius="0.05" length="0.04"/>
+                <cylinder radius="0.031" length="0.025"/>
             </geometry>
             <material name="blue"/>
@@ -89,5 +97,5 @@
         <collision>
             <geometry>
-                <sphere radius="0.05"/>
+                <sphere radius="0.031"/>
             </geometry>
         </collision>
@@ -108,5 +116,5 @@
         <visual>
             <geometry>
-                <sphere radius="0.05"/>
+                <sphere radius="0.051"/>
             </geometry>
             <material name="black"/>
@@ -114,5 +122,5 @@
         <collision>
             <geometry>
-                <sphere radius="0.05"/>
+                <sphere radius="0.051"/>
             </geometry>
         </collision>

Commit message: navigation_stack

File: description/lidar.xacro (robot description, xacro)
@@ -4,5 +4,5 @@
         <parent link="chassis"/>
         <child link="laser_frame"/>
-        <origin xyz="0.1 0 0.075" rpy="0 0 0"/>
+        <origin xyz="0.1 0 0.080" rpy="0 0 0"/>
     </joint>
     <link name="laser_frame">

Commit message: 2022.10.4

File: description/lidar.xacro (robot description, xacro)
@@ -4,10 +4,10 @@
         <parent link="chassis"/>
         <child link="laser_frame"/>
-        <origin xyz="0.1 0 0.080" rpy="0 0 0"/>
+        <origin xyz="0.12 0 0.11" rpy="0 0 0"/>
     </joint>
     <link name="laser_frame">
         <visual>
             <geometry>
-                <cylinder radius="0.05" length="0.04"/>
+                <cylinder radius="0.025" length="0.04"/>
             </geometry>
             <material name="red"/>
@@ -15,5 +15,5 @@
         <collision>
             <geometry>
-                <cylinder radius="0.05" length="0.04"/>
+                <cylinder radius="0.025" length="0.04"/>
             </geometry>
         </collision>

File: description/robot_core.xacro (robot description, xacro)
@@ -38,5 +38,5 @@
             <origin xyz="0.15 0 0.05"/>
             <geometry>
-                <box size="0.23 0.3 0.05"/>
+                <box size="0.15 0.2 0.1"/>
             </geometry>
             <material name="white"/>
@@ -59,5 +59,5 @@
         <parent link="base_link"/>
         <child link="left_wheel"/>
-        <origin xyz="0 0.175 -0.02" rpy="-${pi/2} 0 0" />
+        <origin xyz="0 0.11 -0.02" rpy="-${pi/2} 0 0" />
         <axis xyz="0 0 1"/>
     </joint>
@@ -85,5 +85,5 @@
         <parent link="base_link"/>
         <child link="right_wheel"/>
-        <origin xyz="0 -0.175 -0.02" rpy="${pi/2} 0 0" />
+        <origin xyz="0 -0.11 -0.02" rpy="${pi/2} 0 0" />
         <axis xyz="0 0 -1"/>
     </joint>
@@ -111,10 +111,10 @@
         <parent link="chassis"/>
         <child link="caster_wheel"/>
-        <origin xyz="0.24 0 0"/>
+        <origin xyz="0.2 0 -0.031"/>
     </joint>
     <link name="caster_wheel">
         <visual>
             <geometry>
-                <sphere radius="0.051"/>
+                <sphere radius="0.02"/>
             </geometry>
             <material name="black"/>
@@ -122,8 +122,8 @@
         <collision>
             <geometry>
-                <sphere radius="0.051"/>
+                <sphere radius="0.02"/>
             </geometry>
         </collision>
-        <xacro:inertial_sphere mass="0.1" radius="0.05">
+        <xacro:inertial_sphere mass="0.1" radius="0.02">
             <origin xyz="0 0 0" rpy="0 0 0"/>
         </xacro:inertial_sphere>
